File: pcb/m5stack-rfm95.brd (EAGLE design)
At the start: 50 x 50 mm, 4 parts

Commit message: Changes in the PCB
Parts:
- removed U$3: RFM69HCW-RFM95, xose:RFM69HCW-RFM95-MINPADS
- removed U$4: RFM69CW-MINPADS, xose:RFM69CW-MINPADS
- added IC1: RFM69HCW-RFM95, xose:RFM69HCW-RFM95-MINPADS
- added IC3: UBLOX_MAX7, xose:UBLOX_MAX7
- added JP1: (no value), xose:JST-2-SMD
- added Q1: P-CHANNEL MOSFET, xose:SOT23-R
- added R1: 150, xose:0805
- added R2: 10K, xose:0805
- added R3, R4: 0R, xose:0805
- added R5, R6: 1M, xose:0805
- added X3: (no value), adafruit:SMA90_DIP
- added X4, X5: (no value), adafruit:U.FL
- moved X1 7.80 mm to (32.8, 45.7)
Connections:
- removed net ANT: U$3.ANT, U$4.1, X1.ANTENNA
- new net 3V3_GPS: IC3.P$6, IC3.P$7, IC3.P$8, Q1.3
- new net ANT_GPS: IC3.P$11, R4.2, X5.3
- new net ANT_RF: IC1.ANT, R3.2, X4.3
- new net N$1: R4.1, X1.ANTENNA
- new net N$2: R3.1, X3.ANTENNA
- new net N$3: Q1.1, R1.2
- new net VCC_RF: IC3.P$14
- new net V_ANT: IC3.P$15
- net 3V3: now also IC1.VDD, Q1.2, R2.2; no longer U$3.VDD, U$4.2
- net BAT: now also JP1.1, R5.1
- net G05: now also IC1.NSS; no longer U$3.NSS, U$4.6
- net G15: now also R6.2
- net G16: now also IC1.DIO1; no longer U$3.DIO1
- net G17: now also IC1.DIO2; no longer U$3.DIO2
- net G18: now also IC1.SCK; no longer U$3.SCK, U$4.5
- net G19: now also IC1.MISO; no longer U$3.MISO, U$4.7
- net G21: now also IC3.P$3
- net G22: now also IC3.P$2
- net G23: now also IC1.MOSI; no longer U$3.MOSI, U$4.4
- net G25: now also R1.1, R2.1
- net G26: now also IC1.DIO0; no longer U$3.DIO0, U$4.8
- net G34: now also R5.2, R6.1
- net G36: now also IC1.RESET; no longer U$3.RESET, U$4.10
- net GND: now also IC1.GND, IC1.GND1, IC1.GND2, IC3.P$1, IC3.P$10, IC3.P$12, JP1.2, X3.GND1, X3.GND2, X3.GND3, X3.GND4, X4.1, X4.2, X5.1, X5.2; no longer U$3.GND, U$3.GND1, U$3.GND2, U$4.3, U$4.9
Routing:
- net G21: track 0.00 -> 63.5 mm, vias 0 -> 3
- net G22: track 0.00 -> 60.5 mm, vias 0 -> 3
- net G25: track 0.00 -> 43.3 mm, vias 0 -> 2
- net GND: track 8.67 -> 40.7 mm, vias 5 -> 7
- net 3V3: track 22.5 -> 54.4 mm, vias 0 -> 2
- net G26: track 38.4 -> 18.2 mm, vias 1 -> 0
- net ANT: track 11.1 -> 0.00 mm
- net BAT: track 0.00 -> 10.2 mm
- net ANT_GPS: track 0.00 -> 9.81 mm
- net 3V3_GPS: track 0.00 -> 9.59 mm
- net G15: track 0.00 -> 8.92 mm
- net G05: track 42.3 -> 35.1 mm, vias 4 -> 2
- net G34: track 0.00 -> 7.16 mm
- net ANT_RF: track 0.00 -> 5.45 mm
- net G36: track 40.1 -> 35.3 mm
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Other:
- outline, holes or cut-outs redrawn
- board text added: "Tinkerman 2018 M5STACK RFM95 v0.2.20181030"
- board text removed: "RFM69C"
- board text removed: "Tinkerman 2018 M5STACK RFM69C/RFM95 v0.1.20180330"
