File: pcb/m5stack-rfm95.sch (EAGLE design)
At the start: 4 parts

Commit message: Changes in the PCB
Parts:
- removed U$3: RFM69HCW-RFM95, xose:RFM69HCW-RFM95
- removed U$4: RFM69CW-MINPADS, xose:RFM69CW-MINPADS
- added IC1: RFM69HCW-RFM95, xose:RFM69HCW-RFM95
- added IC3: UBLOX_MAX7, xose:UBLOX_MAX7
- added JP1: (no value), xose:M02-JST-2MM-SMT
- added Q1: P-CHANNEL MOSFET, xose:MOSFET-P
- added R1: 150, xose:RESISTOR0805
- added R2: 10K, xose:RESISTOR0805
- added R3, R4: 0R, xose:RESISTOR0805
- added R5, R6: 1M, xose:RESISTOR0805
- added X3: (no value), adafruit:SMACONNECTOR
- added X4, X5: (no value), adafruit:ANTENNA_U.FL
Connections:
- removed net ANT: U$3.ANT, U$4.ANT, X1.ANT
- new net 3V3_GPS: IC3.VCC, IC3.VCC_IO, IC3.V_BCKP, Q1.D
- new net ANT_GPS: IC3.RF_IN, R4.2, X5.SIGNAL
- new net ANT_RF: IC1.ANT, R3.2, X4.SIGNAL
- new net N$1: R4.1, X1.ANT
- new net N$2: R3.1, X3.ANT
- new net N$3: Q1.G, R1.2
- net 3V3: now also IC1.VCC, Q1.S, R2.2; no longer U$3.VCC, U$4.3.3V
- net BAT: now also JP1.2, R5.1
- net G05: now also IC1.SEL; no longer U$3.SEL, U$4.NSS
- net G15: now also R6.2
- net G16: now also IC1.DIO1; no longer U$3.DIO1
- net G17: now also IC1.DIO2; no longer U$3.DIO2
- net G18: now also IC1.SCK; no longer U$3.SCK, U$4.SCK
- net G19: now also IC1.MISO; no longer U$3.MISO, U$4.MISO
- net G21: now also IC3.RXD
- net G22: now also IC3.TXD
- net G23: now also IC1.MOSI; no longer U$3.MOSI, U$4.MOSI
- net G25: now also R1.1, R2.1
- net G26: now also IC1.DIO0; no longer U$3.DIO0, U$4.DIO0
- net G34: now also R5.2, R6.1
- net G36: now also IC1.RESET; no longer U$3.RESET, U$4.RST
- net GND: now also IC1.GND, IC1.GND1, IC1.GND2, IC3.GND@1, IC3.GND@2, IC3.GND@3, JP1.1, X3.GND1, X3.GND2, X3.GND3, X3.GND4, X4.GND@0, X4.GND@1, X5.GND@0, X5.GND@1; no longer U$3.GND, U$3.GND1, U$3.GND2, U$4.GND@1, U$4.GND@2
Other:
- note added: "BATTERY MONITOR"
- note added: "GPS"
- note removed: "RFM69C RADIO"
- note removed: "SMA CONNECTOR"
- moved on the sheet: U$2, X1
